File: Eagle/satcam_v3_mini.brd (EAGLE design)
At the start: 35.6 x 59.7 mm, 73 parts, among them IC1 24AA64-I/OT, IC2 MCP6001U, IC3 TC1015-2.8VCT, IC4 STM32F446RET6, IC5 TC1015-2.8VCT, IC6 LF50CDT, Q1 FDV301N, Q2 ABM3B-8.000MHZ-10-1-U-T

Commit message: SVN revision 1158
Parts:
- C5, C6: value 15p -> 12p
- R3: value 2k2 -> 680
Connections:
- net SSTV_RX: now also JP1.4, R4.1; no longer JP1.3, R3.1
- net SSTV_TX: now also JP1.3, R3.1; no longer JP1.4, R4.1
Routing:
- net D4: vias 3 -> 2
Changed lines of the file:
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@@
 <text x="16.51" y="58.42" size="0.8128" layer="100" font="vector" ratio="15" align="bottom-center">AUD</text>
 <text x="19.05" y="58.42" size="0.8128" layer="100" font="vector" ratio="15" align="bottom-center">ST</text>
-<text x="21.59" y="58.42" size="0.8128" layer="100" font="vector" ratio="15" align="bottom-center">TXD</text>
-<text x="24.13" y="58.42" size="0.8128" layer="100" font="vector" ratio="15" align="bottom-center">RXD</text>
+<text x="24.13" y="58.42" size="0.8128" layer="100" font="vector" ratio="15" align="bottom-center">TXD</text>
+<text x="21.59" y="58.42" size="0.8128" layer="100" font="vector" ratio="15" align="bottom-center">RXD</text>
 <text x="26.67" y="58.42" size="0.8128" layer="100" font="vector" ratio="15" align="bottom-center">EN</text>
 <text x="29.21" y="58.42" size="0.8128" layer="100" font="vector" ratio="15" align="bottom-center">VDD</text>
@@
 <element name="IC4" library="satcam" package="TQFP64-10X10" value="STM32F446RET6" x="13.335" y="19.05" smashed="yes" rot="R270">
 <attribute name="NAME" x="19.939" y="22.86" size="1.778" layer="25" rot="R270"/>
-<attribute name="VALUE" x="8.001" y="25.2174" size="0.8128" layer="27" font="vector" ratio="12"/>
+<attribute name="VALUE" x="8.636" y="25.2174" size="0.8128" layer="27" font="vector" ratio="12"/>
 </element>
 <element name="IC3" library="satcam" package="SOT23-5" value="TC1015-2.8VCT" x="28.575" y="44.45" smashed="yes" rot="R180">
@@
 <element name="C15" library="rcl" package="C0603" value="100n" x="5.3975" y="23.8125" smashed="yes" rot="R90">
 <attribute name="NAME" x="4.6355" y="22.9235" size="1.27" layer="25" rot="R90"/>
-<attribute name="VALUE" x="3.8735" y="24.9555" size="0.8128" layer="27" font="vector" ratio="12"/>
+<attribute name="VALUE" x="4.5085" y="24.9555" size="0.8128" layer="27" font="vector" ratio="12"/>
 </element>
 <element name="C13" library="rcl" package="C0603" value="100n" x="10.4775" y="27.94" smashed="yes" rot="R90">
@@
 <attribute name="VALUE" x="3.1115" y="16.637" size="0.8128" layer="27" font="vector" ratio="12" rot="R180"/>
 </element>
-<element name="C6" library="rcl" package="C0603" value="15p" x="17.145" y="36.83" smashed="yes" rot="R180">
+<element name="C6" library="rcl" package="C0603" value="12p" x="17.145" y="36.83" smashed="yes" rot="R180">
 <attribute name="NAME" x="18.034" y="36.068" size="1.27" layer="25" rot="R180"/>
 <attribute name="VALUE" x="18.4785" y="36.3855" size="0.8128" layer="27" font="vector" ratio="12"/>
 </element>
-<element name="C5" library="rcl" package="C0603" value="15p" x="20.32" y="33.02" smashed="yes" rot="R270">
+<element name="C5" library="rcl" package="C0603" value="12p" x="20.32" y="33.02" smashed="yes" rot="R270">
 <attribute name="NAME" x="21.082" y="33.909" size="1.27" layer="25" rot="R270"/>
 <attribute name="VALUE" x="19.431" y="34.163" size="0.8128" layer="27" font="vector" ratio="12"/>
@@
 <element name="C3" library="rcl" package="C0603" value="3n3" x="6.985" y="35.56" smashed="yes">
 <attribute name="NAME" x="6.096" y="36.322" size="1.27" layer="25"/>
-<attribute name="VALUE" x="5.6515" y="36.0045" size="0.8128" layer="27" font="vector" ratio="12" rot="R180"/>
+<attribute name="VALUE" x="6.604" y="36.957" size="0.8128" layer="27" font="vector" ratio="12" rot="R180"/>
 </element>
 <element name="C4" library="rcl" package="C0603" value="10n" x="9.525" y="34.925" smashed="yes" rot="R90">
@@
 <element name="R17" library="rcl" package="R0603" value="5k6" x="6.985" y="33.9725" smashed="yes" rot="R180">
 <attribute name="NAME" x="7.874" y="33.0835" size="1.27" layer="25" rot="R180"/>
-<attribute name="VALUE" x="5.6515" y="34.417" size="0.8128" layer="27" font="vector" ratio="12" rot="R180"/>
+<attribute name="VALUE" x="6.731" y="32.258" size="0.8128" layer="27" font="vector" ratio="12"/>
 </element>
 <element name="R18" library="rcl" package="R0603" value="12k" x="5.3975" y="31.4325" smashed="yes" rot="R90">
 <attribute name="NAME" x="4.5085" y="30.5435" size="1.27" layer="25" rot="R90"/>
-<attribute name="VALUE" x="4.699" y="31.877" size="0.8128" layer="27" font="vector" ratio="12" rot="R180"/>
+<attribute name="VALUE" x="6.096" y="30.988" size="0.8128" layer="27" font="vector" ratio="12"/>
 </element>
 <element name="C2" library="rcl" package="C0603" value="47n" x="9.525" y="38.735" smashed="yes" rot="R90">
@@
 <attribute name="VALUE" x="26.289" y="48.387" size="0.8128" layer="27" font="vector" ratio="12" rot="R180"/>
 </element>
-<element name="R3" library="rcl" package="R0603" value="2k2" x="22.86" y="53.34" smashed="yes" rot="R270">
+<element name="R3" library="rcl" package="R0603" value="680" x="22.86" y="53.34" smashed="yes" rot="R270">
 <attribute name="NAME" x="23.749" y="54.229" size="1.27" layer="25" rot="R270"/>
 <attribute name="VALUE" x="21.9075" y="54.2925" size="0.8128" layer="27" font="vector" ratio="12"/>
@@
 <element name="L3" library="satcam" package="R0603" value="FB" x="8.89" y="27.94" smashed="yes" rot="R90">
 <attribute name="NAME" x="8.255" y="27.305" size="1.27" layer="25" rot="R90"/>
-<attribute name="VALUE" x="7.3025" y="29.21" size="0.8128" layer="27" font="vector" ratio="12"/>
+<attribute name="VALUE" x="7.62" y="29.21" size="0.8128" layer="27" font="vector" ratio="12"/>
 </element>
 <element name="L2" library="satcam" package="R0603" value="FB" x="32.0675" y="21.2725" smashed="yes" rot="R90">
@@
 <signal name="D4">
 <contactref element="IC4" pad="52"/>
-<wire x1="17.49" y1="16.8" x2="19.035" y2="16.8" width="0.254" layer="1"/>
-<wire x1="17.4625" y1="16.8275" x2="17.49" y2="16.8" width="0.254" layer="1"/>
-<via x="17.4625" y="16.8275" extent="1-16" drill="0.4"/>
+<wire x1="18.125" y1="16.8" x2="19.035" y2="16.8" width="0.254" layer="1"/>
+<wire x1="18.0975" y1="16.8275" x2="18.125" y2="16.8" width="0.254" layer="1"/>
 <contactref element="CAM1" pad="7"/>
-<wire x1="17.4625" y1="16.8275" x2="13.335" y2="16.8275" width="0.254" layer="1"/>
+<wire x1="18.0975" y1="16.8275" x2="13.335" y2="16.8275" width="0.254" layer="1"/>
 <via x="13.335" y="16.8275" extent="1-16" drill="0.4"/>
 <wire x1="13.335" y1="16.8275" x2="13.97" y2="16.1925" width="0.254" layer="16"/>
@@
 <wire x1="17.145" y1="54.9275" x2="17.145" y2="54.19" width="0.6096" layer="1"/>
 </signal>
-<signal name="SSTV_RX">
+<signal name="SSTV_TX">
 <contactref element="R3" pad="1"/>
 <contactref element="JP1" pad="3"/>
@@
 <wire x1="24.13" y1="55.46" x2="22.86" y2="54.19" width="0.6096" layer="1"/>
 </signal>
-<signal name="SSTV_TX">
+<signal name="SSTV_RX">
 <contactref element="R4" pad="1"/>
 <contactref element="JP1" pad="4"/>

Commit message: SVN revision 1192
Parts:
- added R33: 10k, rcl:R0603
- moved Q1 0.95 mm to (13.7, 50.2)
Connections:
- net GND: now also R33.1
- net GPIO_PTT: now also R33.2
Routing:
- net GPIO_PTT: track 45.5 -> 43.8 mm
- net GND: track 47.3 -> 48.5 mm, vias 94 -> 93
- net N$3: track 2.52 -> 3.04 mm
Other:
- board text added: "OK2ALP v3/2020"
- board text removed: "OK2ALP v3/2019"
Changed lines of the file:
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@@
 <setting verticaltext="up"/>
 </settings>
-<grid distance="0.025" unitdist="inch" unit="mm" style="dots" multiple="1" display="no" altdistance="0.0125" altunitdist="inch" altunit="inch"/>
+<grid distance="0.025" unitdist="inch" unit="mm" style="dots" multiple="1" display="no" altdistance="12.5" altunitdist="mil" altunit="mm"/>
 <layers>
 <layer number="1" name="Top" color="4" fill="1" visible="yes" active="yes"/>
@@
 <layer number="27" name="tValues" color="7" fill="1" visible="yes" active="yes"/>
 <layer number="28" name="bValues" color="7" fill="1" visible="yes" active="yes"/>
-<layer number="29" name="tStop" color="7" fill="3" visible="yes" active="yes"/>
+<layer number="29" name="tStop" color="7" fill="3" visible="no" active="yes"/>
 <layer number="30" name="bStop" color="7" fill="6" visible="no" active="yes"/>
 <layer number="31" name="tCream" color="7" fill="4" visible="no" active="yes"/>
@@
 <wire x1="35.56" y1="3.175" x2="35.56" y2="56.515" width="0.1" layer="20"/>
 <wire x1="0" y1="56.515" x2="0" y2="3.175" width="0.1" layer="20"/>
-<text x="4.1275" y="18.7325" size="1.4224" layer="100" font="vector" ratio="15" rot="R90">OK2ALP v3/2019</text>
+<text x="4.1275" y="18.7325" size="1.4224" layer="100" font="vector" ratio="15" rot="R90">OK2ALP v3/2020</text>
 <text x="32.7025" y="34.6075" size="0.8128" layer="100" font="vector" ratio="15">GND</text>
 <text x="32.7025" y="37.465" size="0.8128" layer="100" font="vector" ratio="15">SW-</text>
@@
 <element name="R12" library="rcl" package="R0603" value="10k" x="20.955" y="50.165" smashed="yes" rot="R90">
 <attribute name="NAME" x="20.066" y="49.276" size="1.27" layer="25" rot="R90"/>
-<attribute name="VALUE" x="20.32" y="48.26" size="0.8128" layer="27" font="vector" ratio="12"/>
+<attribute name="VALUE" x="20.6375" y="48.26" size="0.8128" layer="27" font="vector" ratio="12"/>
 </element>
 <element name="R2" library="rcl" package="R0603" value="680" x="17.145" y="53.34" smashed="yes" rot="R270">
@@
 <element name="R14" library="rcl" package="R0603" value="10k" x="19.05" y="50.165" smashed="yes" rot="R90">
 <attribute name="NAME" x="18.415" y="49.53" size="1.27" layer="25" rot="R90"/>
-<attribute name="VALUE" x="17.78" y="48.26" size="0.8128" layer="27" font="vector" ratio="12"/>
+<attribute name="VALUE" x="18.0975" y="48.26" size="0.8128" layer="27" font="vector" ratio="12"/>
 </element>
 <element name="JP1" library="pinhead" package="1X10" value="" x="17.78" y="56.515" smashed="yes" rot="R180">
@@
 <attribute name="VALUE" x="30.48" y="59.69" size="1.27" layer="27" rot="R180"/>
 </element>
-<element name="Q1" library="transistor-small-signal" package="SOT23" value="FDV301N" x="14.605" y="50.165" smashed="yes" rot="R90">
-<attribute name="NAME" x="12.7" y="48.26" size="1.27" layer="25" rot="R90"/>
-<attribute name="VALUE" x="13.0175" y="48.26" size="0.8128" layer="27" font="vector" ratio="12" rot="R90"/>
+<element name="Q1" library="transistor-small-signal" package="SOT23" value="FDV301N" x="13.6525" y="50.165" smashed="yes" rot="R90">
+<attribute name="NAME" x="11.7475" y="48.26" size="1.27" layer="25" rot="R90"/>
+<attribute name="VALUE" x="12.22375" y="49.05375" size="0.8128" layer="27" font="vector" ratio="12" rot="R90"/>
 </element>
 <element name="R26" library="rcl" package="R0603" value="47k" x="8.89" y="45.085" smashed="yes">
@@
 <attribute name="NAME" x="9.89" y="46.115" size="1.016" layer="25" rot="R180"/>
 <attribute name="VALUE" x="7.6675" y="47.3025" size="0.8128" layer="27" font="vector" ratio="12" rot="R180"/>
+</element>
+<element name="R33" library="rcl" package="R0603" value="10k" x="16.51" y="50.165" smashed="yes" rot="R270">
+<attribute name="NAME" x="17.145" y="50.8" size="1.27" layer="25" rot="R270"/>
+<attribute name="VALUE" x="15.5575" y="48.26" size="0.8128" layer="27" font="vector" ratio="12"/>
 </element>
 </elements>
@@
 <wire x1="34.925" y1="46.99" x2="34.6075" y2="47.3075" width="0.254" layer="1"/>
 <wire x1="34.6075" y1="47.3075" x2="33.9725" y2="47.3075" width="0.254" layer="1"/>
-<via x="16.8275" y="50.8" extent="1-16" drill="0.4"/>
+<via x="15.5575" y="51.7525" extent="1-16" drill="0.4"/>
 <via x="12.065" y="21.2725" extent="1-16" drill="0.4"/>
 <via x="8.255" y="1.27" extent="1-16" drill="0.4"/>
@@
 <via x="2.8575" y="45.72" extent="1-16" drill="0.4"/>
 <via x="7.62" y="50.165" extent="1-16" drill="0.4"/>
-<via x="12.3825" y="53.34" extent="1-16" drill="0.4"/>
 <via x="22.86" y="50.4825" extent="1-16" drill="0.4"/>
 <via x="20.955" y="47.9425" extent="1-16" drill="0.4"/>
@@
 <wire x1="31.115" y1="13.335" x2="30.1625" y2="12.3825" width="0.4064" layer="1"/>
 <wire x1="30.1625" y1="12.3825" x2="30.1625" y2="12.065" width="0.4064" layer="1"/>
+<contactref element="R33" pad="1"/>
+<wire x1="15.5575" y1="51.7525" x2="15.5575" y2="51.435" width="0.254" layer="1"/>
+<wire x1="15.5575" y1="51.435" x2="15.24" y2="51.1175" width="0.254" layer="1"/>
+<wire x1="15.24" y1="51.1175" x2="14.755" y2="51.1175" width="0.254" layer="1"/>
+<wire x1="14.755" y1="51.1175" x2="14.7525" y2="51.115" width="0.254" layer="1"/>
 </signal>
 <signal name="VCC">
@@
 <contactref element="R2" pad="2"/>
 <wire x1="9.525" y1="39.585" x2="9.525" y2="40.3225" width="0.254" layer="1"/>
-<via x="17.4625" y="51.7525" extent="1-16" drill="0.4"/>
-<wire x1="17.145" y1="52.49" x2="17.145" y2="52.07" width="0.254" layer="1"/>
-<wire x1="17.145" y1="52.07" x2="17.4625" y2="51.7525" width="0.254" layer="1"/>
+<via x="17.78" y="51.7525" extent="1-16" drill="0.4"/>
+<wire x1="17.145" y1="52.49" x2="17.145" y2="52.3875" width="0.254" layer="1"/>
+<wire x1="17.145" y1="52.3875" x2="17.78" y2="51.7525" width="0.254" layer="1"/>
 <via x="9.525" y="40.3225" extent="1-16" drill="0.4"/>
-<wire x1="17.4625" y1="51.7525" x2="18.415" y2="50.8" width="0.254" layer="16"/>
-<wire x1="18.415" y1="50.8" x2="18.415" y2="49.53" width="0.254" layer="16"/>
+<wire x1="17.78" y1="51.7525" x2="18.415" y2="51.1175" width="0.254" layer="16"/>
+<wire x1="18.415" y1="51.1175" x2="18.415" y2="49.53" width="0.254" layer="16"/>
 <wire x1="18.415" y1="49.53" x2="17.78" y2="48.895" width="0.254" layer="16"/>
 <wire x1="17.78" y1="48.895" x2="11.7475" y2="48.895" width="0.254" layer="16"/>
@@
 <via x="4.445" y="20.32" extent="1-16" drill="0.4"/>
 <contactref element="Q1" pad="1"/>
-<wire x1="15.705" y1="49.215" x2="16.83" y2="49.215" width="0.254" layer="1"/>
-<wire x1="16.83" y1="49.215" x2="17.4625" y2="49.8475" width="0.254" layer="1"/>
-<via x="17.4625" y="49.8475" extent="1-16" drill="0.4"/>
-<wire x1="17.4625" y1="49.8475" x2="17.145" y2="49.53" width="0.254" layer="16"/>
-<wire x1="17.145" y1="49.53" x2="11.43" y2="49.53" width="0.254" layer="16"/>
+<via x="15.5575" y="49.8475" extent="1-16" drill="0.4"/>
+<wire x1="15.5575" y1="49.8475" x2="15.24" y2="49.53" width="0.254" layer="16"/>
+<wire x1="15.24" y1="49.53" x2="11.43" y2="49.53" width="0.254" layer="16"/>
 <wire x1="11.43" y1="49.53" x2="2.54" y2="40.64" width="0.254" layer="16"/>
+<contactref element="R33" pad="2"/>
+<wire x1="14.7525" y1="49.215" x2="14.925" y2="49.215" width="0.254" layer="1"/>
+<wire x1="14.925" y1="49.215" x2="15.5575" y2="49.8475" width="0.254" layer="1"/>
+<wire x1="16.51" y1="49.315" x2="16.09" y2="49.315" width="0.254" layer="1"/>
+<wire x1="16.09" y1="49.315" x2="15.5575" y2="49.8475" width="0.254" layer="1"/>
 </signal>
 <signal name="UART2TX">
@@
 <contactref element="R6" pad="2"/>
 <contactref element="Q1" pad="3"/>
-<wire x1="13.505" y1="50.165" x2="13.505" y2="50.97" width="0.254" layer="1"/>
-<wire x1="13.505" y1="50.97" x2="13.97" y2="51.435" width="0.254" layer="1"/>
-<wire x1="13.97" y1="51.435" x2="13.97" y2="52.49" width="0.254" layer="1"/>
+<wire x1="13.97" y1="52.49" x2="13.755" y2="52.49" width="0.254" layer="1"/>
+<wire x1="13.755" y1="52.49" x2="12.5525" y2="51.2875" width="0.254" layer="1"/>
+<wire x1="12.5525" y1="50.165" x2="12.5525" y2="51.2875" width="0.254" layer="1"/>
 </signal>
 <signal name="N$6">
