File: Eagle/satcam_v3_mini.sch (EAGLE design)
At the start: 73 parts, among them IC1 24AA64-I/OT, IC2 MCP6001U, IC3 TC1015-2.8VCT, IC4 STM32F446RET6, IC5 TC1015-2.8VCT, IC6 LF50CDT, Q1 FDV301N, Q2 ABM3B-8.000MHZ-10-1-U-T

Commit message: SVN revision 1158
Parts:
- C5, C6: value 15p -> 12p
- R3: value 2k2 -> 680
Connections:
- net SSTV_RX: now also JP1.4, R4.1; no longer JP1.3, R3.1
- net SSTV_TX: now also JP1.3, R3.1; no longer JP1.4, R4.1
Changed lines of the file:
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@@
 <part name="C14" library="rcl" deviceset="C-EU" device="C0603" value="4u7"/>
 <part name="GND24" library="supply1" deviceset="GND" device=""/>
-<part name="C6" library="rcl" deviceset="C-EU" device="C0603" value="15p"/>
-<part name="C5" library="rcl" deviceset="C-EU" device="C0603" value="15p"/>
+<part name="C6" library="rcl" deviceset="C-EU" device="C0603" value="12p"/>
+<part name="C5" library="rcl" deviceset="C-EU" device="C0603" value="12p"/>
 <part name="IC2" library="satcam" deviceset="MCP6001U" device=""/>
 <part name="C10" library="rcl" deviceset="C-EU" device="C0603" value="100n"/>
@@
 <part name="R10" library="rcl" deviceset="R-EU_" device="R0603" value="100k"/>
 <part name="GND4" library="supply1" deviceset="GND" device=""/>
-<part name="R3" library="rcl" deviceset="R-EU_" device="R0603" value="2k2"/>
+<part name="R3" library="rcl" deviceset="R-EU_" device="R0603" value="680"/>
 <part name="R4" library="rcl" deviceset="R-EU_" device="R0603" value="2k2"/>
 <part name="R6" library="rcl" deviceset="R-EU_" device="R0603" value="47"/>
@@
 </segment>
 </net>
-<net name="SSTV_RX" class="0">
+<net name="SSTV_TX" class="0">
 <segment>
 <wire x1="40.64" y1="124.46" x2="20.32" y2="124.46" width="0.1524" layer="91"/>
@@
 </segment>
 </net>
-<net name="SSTV_TX" class="0">
+<net name="SSTV_RX" class="0">
 <segment>
 <wire x1="40.64" y1="121.92" x2="20.32" y2="121.92" width="0.1524" layer="91"/>

Commit message: SVN revision 1192
Parts:
- added R33: 10k, rcl:R-EU_R0603
Connections:
- net GND: now also R33.1
- net GPIO_PTT: now also R33.2
Changed lines of the file:
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@@
 <part name="GND39" library="supply1" deviceset="GND" device=""/>
 <part name="VDD1" library="supply1" deviceset="VDD" device=""/>
+<part name="R33" library="rcl" deviceset="R-EU_" device="R0603" value="10k"/>
+<part name="GND38" library="supply1" deviceset="GND" device=""/>
 </parts>
 <sheets>
@@
 <instance part="JP1" gate="A" x="50.8" y="33.02"/>
 <instance part="Q1" gate="G$1" x="88.9" y="81.28" rot="MR0"/>
-<instance part="GND13" gate="1" x="88.9" y="73.66"/>
+<instance part="GND13" gate="1" x="88.9" y="63.5"/>
 <instance part="R26" gate="G$1" x="121.92" y="38.1"/>
 <instance part="R25" gate="G$1" x="111.76" y="27.94" rot="R90"/>
@@
 <instance part="GND39" gate="1" x="144.78" y="17.78"/>
 <instance part="VDD1" gate="G$1" x="40.64" y="66.04" rot="MR0"/>
+<instance part="R33" gate="G$1" x="101.6" y="71.12" rot="R90"/>
+<instance part="GND38" gate="1" x="101.6" y="63.5"/>
 </instances>
 <busses>
@@
 <pinref part="Q1" gate="G$1" pin="S"/>
 <pinref part="GND13" gate="1" pin="GND"/>
+<wire x1="88.9" y1="66.04" x2="88.9" y2="76.2" width="0.1524" layer="91"/>
 </segment>
 <segment>
@@
 <pinref part="C26" gate="G$1" pin="2"/>
 <wire x1="144.78" y1="20.32" x2="144.78" y2="22.86" width="0.1524" layer="91"/>
+</segment>
+<segment>
+<pinref part="R33" gate="G$1" pin="1"/>
+<pinref part="GND38" gate="1" pin="GND"/>
 </segment>
 </net>
@@
 <label x="111.76" y="78.74" size="1.778" layer="95"/>
 <pinref part="Q1" gate="G$1" pin="G"/>
-<wire x1="93.98" y1="78.74" x2="127" y2="78.74" width="0.1524" layer="91"/>
-</segment>
-<segment>
+<wire x1="93.98" y1="78.74" x2="101.6" y2="78.74" width="0.1524" layer="91"/>
+<pinref part="R33" gate="G$1" pin="2"/>
+<wire x1="101.6" y1="78.74" x2="127" y2="78.74" width="0.1524" layer="91"/>
+<wire x1="101.6" y1="76.2" x2="101.6" y2="78.74" width="0.1524" layer="91"/>
+<junction x="101.6" y="78.74"/>
+</segment>
+<segment>
