File: Eagle/satcam_v4_pocket_revB.sch (EAGLE design)
At the start: 74 parts, among them IC1 24AA64-I/OT, IC2 MCP6001U, IC3 TC1015-2.8VCT, IC4 STM32F446RET6, IC5 TC1015-2.8VCT, IC6 LF50CDT, Q1 FDV301N, Q2 ABM3B-8.000MHZ-10-1-U-T

Commit message: SVN revision 1250
Parts:
- removed C26: 10u/16V, rcl:C-EUC0805K
- removed JP1: (no value), pinhead:PINHD-1X10
- removed JP2: DEBUG, pinhead:PINHD-1X6
- removed Q1: FDV301N, transistor-small-signal:BSS123
- removed R11, R13, R33: 10k, rcl:R-EU_R0603
- removed R3: 680, rcl:R-EU_R0603
- removed R32: 1R, rcl:R-EU_R0603
- removed R4, R5: 2k2, rcl:R-EU_R0603
- removed R6: 47, rcl:R-EU_R0603
- removed R8, R9: 8k2, rcl:R-EU_R0603
- added C24, C28, C32: 100n, rcl:C-EUC0603
- added C31: 10n, rcl:C-EUC0603
- added D1: GL5549, satcam:SFH229
- added IC8: 24AA64-I/OT, satcam:24AA64-I/OT
- added P1: 53398-0610, con-molex-picoblade:53398-0610
- added Q3, Q4, Q5, Q7: FDV301N, transistor-small-signal:BSS123
- added TP1, TP2, TP3, TP4, TP5: TPB1,27, testpad:TPB1,27
- added U$1, U$2, U$3, U$4: MOUNT_HOLE2, satcam:MOUNT_HOLE2
- C2: value 47n -> 100n
- C25: value 10u/16V -> 1u; device rcl:C-EUC0805K -> rcl:C-EUC0603
- IC6: value LF50CDT -> M25P16; device linear:7805DT -> satcam:M25P16
- R10: value 100k -> 47k
- R12: value 10k -> 47k
- R19, R21, R22: value 47 -> 10k
- R20: value 47 -> 470
- R31: value DNP -> 10k
- R7: value 8k2 -> 10k
Connections:
- removed net +5V: C25.1, C7.1, IC3.IN, IC6.VO, L2.2, R31.2
- removed net AUDIO: JP1.6, R1.2, R2.1
- removed net ENABLE: JP1.2, R5.1
- removed net GPIO_M0: IC4.PC5/USART3_RX, R11.2, R9.2
- removed net GPIO_M1: IC4.PC10/USART3_TX, R13.2, R8.2
- removed net GPIO_PTT: IC4.PC4, Q1.G, R33.2
- removed net GPIO_START: IC4.PA1, R14.2, R7.2
- removed net MODE0: JP1.9, R9.1
- removed net MODE1: JP1.8, R8.1
- removed net N$137: JP2.4, R20.1
- removed net N$138: JP2.2, R19.1
- removed net N$143: JP2.5, R21.1
- removed net N$145: JP2.6, R22.1
- removed net N$3: Q1.D, R6.2
- removed net N$6: C25.2, R32.2
- removed net PTT: JP1.7, R6.1
- removed net SSTV_RX: JP1.4, R4.1
- removed net SSTV_TX: JP1.3, R3.1
- removed net START: JP1.5, R7.1
- removed net SWO: IC4.PB3/SWO, R22.2
- removed net SYS_SHDN: IC3.EN, R10.2, R5.2
- removed net UART2RX: IC4.PA3/USART2_RX, R12.2, R4.2
- removed net UART2TX: IC4.PA2/USART2_TX, R3.2
- new net AUDIO_ADC: C28.2, IC4.PA7, R10.1, R12.2
- new net AUDIO_IN: C28.1, P1.6
- new net AUDIO_OUT: P1.5, R1.2, R2.1
- new net MISO: IC4.PC2/SPI2_MISO, IC6.DQ1
- new net MOSI: IC4.PC3/SPI2_MOSI, IC6.DQ0
- new net N$14: Q7.D, R19.1
- new net N$15: Q3.D, R20.1
- new net NSS: IC4.PB12/SPI2_NSS, IC6.S, R31.2
- new net SCK: IC4.PB13/SPI2_SCK, IC6.C
- new net SCL1: IC4.PB10/SCL, IC4.PC10/USART3_TX, IC8.SCL, Q5.S, R7.1
- new net SCL2: P1.3, Q5.D, R21.1
- new net SDA1: IC4.PC12/SDA, IC8.SDA, Q4.S, R14.1
- new net SDA2: P1.2, Q4.D, R22.1
- new net SENS_ADC: C31.1, D1.A, IC4.PA0/WKUP0, R19.2, R20.2
- new net SENS_RNG1: IC4.PC0, Q7.G
- new net SENS_RNG2: IC4.PC1, Q3.G
- net ADC_VDD: now also IC4.PB0; no longer IC4.PA0/WKUP0
- net CAM_SCL: now also IC4.PB5; no longer IC4.PB10/SCL
- net CAM_SDA: now also IC4.PB4; no longer IC4.PC12/SDA
- net GND: now also C24.2, C25.2, C31.2, C32.2, IC8.GND, IC8.WP, P1.4, Q3.S, Q7.S, TP4.TP; no longer C26.2, JP1.10, JP2.3, Q1.S, R10.1, R11.1, R13.1, R14.1, R32.1, R33.1
- net LED_G: now also IC4.PB14; no longer IC4.PB1
- net LED_R: now also IC4.PB15; no longer IC4.PB0
- net N$7: now also P1.1; no longer JP1.1
- net NRST: now also TP3.TP; no longer R21.2
- net SWCLK: now also TP1.TP; no longer R19.2
- net SWDIO: now also TP2.TP; no longer R20.2
- net VCC: now also C24.1, C25.1, C32.1, D1.C, IC6.HOLD, IC6.VCC, IC6.W, IC8.VCC, Q4.G, Q5.G, R10.2, R14.2, R31.1, R7.2, TP5.TP; no longer JP2.1
- net VDD: now also C7.1, IC3.EN, IC3.IN, L2.2, R21.2, R22.2; no longer C26.1, IC6.VI, R31.1
Other:
- note added: "(c) 2015-2020 OK2ALP"
- note added: "SatCam - SSTV Camera Module"
- note added: "dummy"
- note added: "v4"
- note removed: "(c) 2015-2019 OK2ALP"
- note removed: "3V3 levels: 2k2 | 10k"
- note removed: "5V levels: 8k2 | 10k"
- note removed: "SatCam - Camera Module for PSAT-2"
- note removed: "v3"
- moved on the sheet: C11, C12, C19, C2, C20, C21, C22, C23, C25, C3, C4, CAM1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
